File: Controller/pcbDesigns/549-anamdev-forceSensor.sch (EAGLE design)
At the start: 42 parts, among them IC1 REG1117, J2 AVR_SPI_PROG_3X2PTH, J3 POWER_JACK, Q1 MMBT4403, U1 328P, U2 HX711

Commit message: added multiple amplifiers for force sensor
Parts:
- removed C15: .1 uF, rcl:C-USC1206
- removed C16: 10uF, rcl:C-USC1206
- removed C17, C18, C8: 0.1uF, rcl:C-USC1206
- removed R11, R12: 100, rcl:R-US_R1206
- removed R13: 10K, rcl:R-US_R1206
- removed R6: 20k, rcl:R-US_R1206
- removed R7: 8.2k, rcl:R-US_R1206
- added C21, C22, C23, C24, C26, C28, C29: 0.1uF, rcl:C-USC1206
- added C25, C27: 10uF, rcl:C-USC1206
- added JP1: (no value), SparkFun-Connectors:M02PTH
- added JP3, JP5: LL, SparkFun-Connectors:M03PTH
- added JP6: LR, SparkFun-Connectors:M03PTH
- added L2: 3.3uH, SparkFun-Passives:INDUCTOR0805-IND
- added Q2: MMBT4403, SparkFun-DiscreteSemi:TRANSISTOR_PNPMMBT4403
- added R14: 20k, rcl:R-US_R1206
- added R15: 8.2k, rcl:R-US_R1206
- added R16, R23: 10k, rcl:R-US_R1206
- added R17, R18, R21, R22: 100, rcl:R-US_R1206
- added R19, R20: 330, rcl:R-US_R1206
- added U8: HX711, Testing:HX711HX711
- C19: value 10uF -> 0.1uF
- C20: value 0.1uF -> 10uF
- JP4: value (none) -> LR; device SparkFun-Connectors:M05PTH -> SparkFun-Connectors:M03PTH
Connections:
- removed net A+: JP4.2, R12.2
- removed net A-: JP4.3, R11.2
- removed net AVDD: C15.1, C16.1, JP4.5, L1.1
- removed net B+: JP2.1, U2.INB+
- removed net B-: JP2.2, U2.INB-
- new net A+0: JP5.2, R18.2
- new net A+1: JP3.2, R22.2
- new net A-0: JP6.2, R17.1
- new net A-1: JP4.2, R21.2
- new net AVDD0: C19.1, C20.1, JP5.3, JP6.3, L1.1
- new net AVDD1: C26.1, C27.1, JP3.3, JP4.3, L2.1
- new net B+0: JP2.1, U8.INB+
- new net B+1: JP1.1, U2.INB+
- new net B-0: JP2.2, U8.INB-
- new net B-1: JP1.2, U2.INB-
- new net N$13: C21.2, U8.VBG
- new net N$16: L1.2, Q2.C, R14.2, U8.AVDD
- new net N$19: C22.2, R18.1, U8.INA+
- new net N$6: Q2.B, U8.BASE
- new net N$8: R14.1, R15.2, U8.VFB
- new net PC0: SL2.3, U1.PC0(ADC0), U8.DOUT
- new net PC1: SL2.4, U1.PC1(ADC1), U2.DOUT
- net GND: now also C20.2, C21.1, C23.2, C24.2, C25.2, C26.2, C27.2, C29.1, JP3.1, JP5.1, JP6.1, R15.1, R20.1, U8.AGND, U8.XI; no longer C15.2, C16.2, C17.2, C18.2, C8.1, JP4.4, R7.1
- net N$17: now also R16.1, U8.RATE; no longer SL2.4, U1.PC1(ADC1)
- net N$18: now also C22.1, R17.2, U8.INA-; no longer SL2.3, U1.PC0(ADC0)
- net N$23: now also R19.1, R20.2; no longer R6.1, R7.2
- net N$24: now also C29.2; no longer C8.2
- net N$25: now also L2.2, R19.2; no longer L1.2, R6.2
- net N$26: now also R23.1; no longer R13.2
- net N$27: now also C28.1, R21.1; no longer C20.1, R11.1
- net N$28: now also C28.2, R22.1; no longer C20.2, R12.1
- net PC2: no longer U2.DOUT
- net SCK: now also U8.PD_SCK
- net VCC: now also C23.1, C24.1, C25.1, Q2.E, R16.2, R23.2, U8.DVDD, U8.VSUP; no longer C17.1, C18.1, C19.1, R13.1
Other:
- note added: "+/WHT"
- note added: "-/BLK"
- note added: "C/RED"
- note added: "Green"
- note added: "IO: 2.7-5.5V"
- note added: "Load Cell headers"
- note added: "VCC: 2.7-5.5V"
- note added: "VDD: 2.7-5.5V"
- note removed: "Alex Wende"
- note removed: "Common Load Cell Colors:"
- note removed: "Green or Blue"
- note removed: "N. Seidle"
- note removed: "Open jumper to set to 80SPS Increases noise per read"
- note removed: "v11"

Commit message: updated pcb boards
Changed lines of the file:
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@@
-</segment>
-</net>
-<net name="N$13" class="0">
-<segment>
-<pinref part="U8" gate="U1" pin="VBG"/>
-<wire x1="162.56" y1="111.76" x2="154.94" y2="111.76" width="0.1524" layer="91"/>
-<wire x1="154.94" y1="111.76" x2="154.94" y2="106.872121875" width="0.1524" layer="91"/>
-<pinref part="C21" gate="G$1" pin="2"/>
-<wire x1="152.51485625" y1="106.872121875" x2="154.94" y2="106.872121875" width="0.1524" layer="91"/>
-<wire x1="154.94" y1="106.872121875" x2="154.94" y2="106.68" width="0.1524" layer="91"/>
 </segment>
 </net>
@@
 <segment>
 <label x="119.38" y="17.78" size="1.778" layer="95"/>
-<pinref part="L2" gate="G$1" pin="1"/>
-<wire x1="147.32" y1="17.78" x2="154.94" y2="17.78" width="0.2032" layer="91"/>
 <pinref part="JP3" gate="G$1" pin="3"/>
 <wire x1="88.9" y1="-76.2" x2="88.9" y2="-71.12" width="0.1524" layer="91"/>
@@
 <wire x1="111.76" y1="-71.12" x2="88.9" y2="-71.12" width="0.1524" layer="91"/>
 <junction x="88.9" y="-71.12"/>
-<wire x1="147.32" y1="17.78" x2="137.352121875" y2="17.78" width="0.1524" layer="91"/>
-<wire x1="137.16" y1="17.78" x2="88.9" y2="17.78" width="0.1524" layer="91"/>
 <wire x1="88.9" y1="17.78" x2="88.9" y2="-71.12" width="0.1524" layer="91"/>
+<pinref part="L2" gate="G$1" pin="1"/>
+<wire x1="147.32" y1="17.78" x2="154.94" y2="17.78" width="0.2032" layer="91"/>
 <pinref part="C27" gate="G$1" pin="1"/>
 <wire x1="147.512121875" y1="15.12514375" x2="147.32" y2="15.12514375" width="0.1524" layer="91"/>
 <wire x1="147.32" y1="15.12514375" x2="147.32" y2="17.78" width="0.1524" layer="91"/>
+<pinref part="C26" gate="G$1" pin="1"/>
+<wire x1="137.352121875" y1="15.12514375" x2="137.16" y2="15.12514375" width="0.1524" layer="91"/>
+<wire x1="137.16" y1="15.12514375" x2="137.16" y2="17.78" width="0.1524" layer="91"/>
+<wire x1="137.16" y1="17.78" x2="147.32" y2="17.78" width="0.1524" layer="91"/>
 <junction x="147.32" y="17.78"/>
-<pinref part="C26" gate="G$1" pin="1"/>
-<wire x1="137.16" y1="17.78" x2="137.352121875" y2="17.78" width="0.1524" layer="91"/>
-<wire x1="137.352121875" y1="17.78" x2="137.352121875" y2="15.12514375" width="0.1524" layer="91"/>
+<wire x1="137.16" y1="17.78" x2="88.9" y2="17.78" width="0.1524" layer="91"/>
+<junction x="137.16" y="17.78"/>
 </segment>
 </net>
@@
 <pinref part="R19" gate="G$1" pin="1"/>
 <pinref part="R20" gate="G$1" pin="2"/>
-</segment>
-</net>
-<net name="N$24" class="0">
-<segment>
-<pinref part="U2" gate="U1" pin="VBG"/>
-<wire x1="200.66" y1="-7.62" x2="193.04" y2="-7.62" width="0.1524" layer="91"/>
-<wire x1="193.04" y1="-7.62" x2="193.04" y2="-12.507878125" width="0.1524" layer="91"/>
-<pinref part="C29" gate="G$1" pin="2"/>
-<wire x1="190.61485625" y1="-12.507878125" x2="193.04" y2="-12.507878125" width="0.1524" layer="91"/>
-<wire x1="193.04" y1="-12.507878125" x2="193.04" y2="-12.7" width="0.1524" layer="91"/>
 </segment>
 </net>
@@
 <segment>
 <label x="81.28" y="137.16" size="1.778" layer="95"/>
-<pinref part="L1" gate="G$1" pin="1"/>
-<wire x1="109.22" y1="137.16" x2="116.84" y2="137.16" width="0.2032" layer="91"/>
 <pinref part="JP5" gate="G$1" pin="3"/>
-<wire x1="109.22" y1="137.16" x2="99.252121875" y2="137.16" width="0.1524" layer="91"/>
-<wire x1="99.252121875" y1="137.16" x2="50.8" y2="137.16" width="0.1524" layer="91"/>
 <wire x1="50.8" y1="137.16" x2="50.8" y2="48.26" width="0.1524" layer="91"/>
 <pinref part="JP6" gate="G$1" pin="3"/>
@@
 <wire x1="73.66" y1="48.26" x2="50.8" y2="48.26" width="0.1524" layer="91"/>
 <junction x="50.8" y="48.26"/>
+<pinref part="L1" gate="G$1" pin="1"/>
+<pinref part="C20" gate="G$1" pin="1"/>
+<wire x1="109.412121875" y1="137.16" x2="109.412121875" y2="134.50514375" width="0.1524" layer="91"/>
+<wire x1="109.22" y1="137.16" x2="109.412121875" y2="137.16" width="0.1524" layer="91"/>
+<wire x1="109.22" y1="137.16" x2="116.84" y2="137.16" width="0.2032" layer="91"/>
+<wire x1="50.8" y1="137.16" x2="99.06" y2="137.16" width="0.1524" layer="91"/>
+<junction x="109.22" y="137.16"/>
 <pinref part="C19" gate="G$1" pin="1"/>
-<wire x1="99.252121875" y1="137.16" x2="99.252121875" y2="134.50514375" width="0.1524" layer="91"/>
-<pinref part="C20" gate="G$1" pin="1"/>
-<wire x1="109.22" y1="137.16" x2="109.412121875" y2="137.16" width="0.1524" layer="91"/>
-<wire x1="109.412121875" y1="137.16" x2="109.412121875" y2="134.50514375" width="0.1524" layer="91"/>
-<junction x="109.22" y="137.16"/>
+<wire x1="99.06" y1="137.16" x2="109.22" y2="137.16" width="0.1524" layer="91"/>
+<wire x1="99.252121875" y1="134.50514375" x2="99.06" y2="134.50514375" width="0.1524" layer="91"/>
+<wire x1="99.06" y1="134.50514375" x2="99.06" y2="137.16" width="0.1524" layer="91"/>
+<junction x="99.06" y="137.16"/>
 </segment>
 </net>
@@
 </segment>
 </net>
+<net name="N$13" class="0">
+<segment>
+<pinref part="U8" gate="U1" pin="VBG"/>
+<pinref part="C21" gate="G$1" pin="2"/>
+<wire x1="162.56" y1="111.76" x2="152.51485625" y2="111.76" width="0.1524" layer="91"/>
+<wire x1="152.51485625" y1="111.76" x2="152.51485625" y2="106.872121875" width="0.1524" layer="91"/>
+</segment>
+</net>
+<net name="N$24" class="0">
+<segment>
+<pinref part="U2" gate="U1" pin="VBG"/>
+<pinref part="C29" gate="G$1" pin="2"/>
+<wire x1="200.66" y1="-7.62" x2="190.61485625" y2="-7.62" width="0.1524" layer="91"/>
+<wire x1="190.61485625" y1="-7.62" x2="190.61485625" y2="-12.507878125" width="0.1524" layer="91"/>
+</segment>
+</net>
